File: SimpleArduinoVlfRadio/Signal Generator.sch (KiCad schematic (older format))
At the start: 20 parts

Commit message: Enable/Disable 555
Allow a digital input to enable/disable the 555 timer. This version only works if the microcontroller operates at 5V (not 3.3V)
Connections:
- net +5V: no longer U?.4 (RESET)
- new net Enable555: U?.4 (RESET)
Changed lines of the file:
@@
 $EndComp
-Wire Wire Line
-	5200 3500 5100 3500
-Wire Wire Line
-	5100 3300 5200 3300
 Wire Wire Line
 	5200 3900 5100 3900
@@
 	1    0    0    -1
 $EndComp
-Wire Wire Line
-	5100 3300 5100 3500
-Connection ~ 5100 3300
 Wire Wire Line
 	4700 3300 4700 3350
@@
 $EndComp
 Wire Wire Line
-	4900 3300 5100 3300
-Wire Wire Line
 	4900 3300 4700 3300
 Connection ~ 4900 3300
@@
 Text HLabel 10350 3500 2    50   Input ~ 0
 FmOut
+Wire Wire Line
+	4900 3300 5200 3300
+Text HLabel 5100 2700 2    50   Input ~ 0
+Enable555
+Wire Wire Line
+	5200 3500 5100 3500
+Wire Wire Line
+	5100 3500 5100 2700
 $EndSCHEMATC

Commit message: Update to working but inefficient design
Design is working well. Need big caps on power for filter and bigger cap for amp. Also need to make sure gain of 10x or more on lm1875. Current draw of 250mA on transmit. Power of 17mA with amplifier disconnected.
Parts:
- C? (x2): value 10u -> 1000u
Connections:
- net at U?.3 (OP_OUT): now also U?.4 (OP_IN-)
Changed lines of the file:
@@
 $Descr A4 11693 8268
 encoding utf-8
-Sheet 2 4
+Sheet 2 5
 Title "Signal Generator"
 Date ""
@@
 P 9550 3950
 F 0 "C?" H 9665 3996 50  0000 L CNN
-F 1 "10u" H 9665 3905 50  0000 L CNN
+F 1 "1000u" H 9665 3905 50  0000 L CNN
 F 2 "" H 9550 3950 50  0001 C CNN
 F 3 "~" H 9550 3950 50  0001 C CNN
@@
 P 10000 3950
 F 0 "C?" H 10115 3996 50  0000 L CNN
-F 1 "10u" H 10115 3905 50  0000 L CNN
+F 1 "1000u" H 10115 3905 50  0000 L CNN
 F 2 "" H 10000 3950 50  0001 C CNN
 F 3 "~" H 10000 3950 50  0001 C CNN
@@
 Wire Wire Line
 	5100 3500 5100 2700
+Wire Wire Line
+	7750 3500 7650 3500
+Wire Wire Line
+	7650 3500 7650 3700
+Wire Wire Line
+	7650 3700 7750 3700
 $EndSCHEMATC

Commit message: Updated Transmitter and finished fsk receiver
Parts:
- U2: renamed from U?; value TLC555CP -> 555; footprint P0008A -> (none)
- U3: renamed from U?; value MAX292-Custom_Library -> MAX292
- gave numbers to parts that had none: 1
Changed lines of the file:
@@
 $Descr A4 11693 8268
 encoding utf-8
-Sheet 2 10
+Sheet 2 14
 Title "Signal Generator"
 Date ""
@@
 Comment4 ""
 $EndDescr
-$Comp
-L Amplifier_Operational:LM358 U?
-U 1 1 616F9E75
-P 3400 3550
-AR Path="/616F9E75" Ref="U?"  Part="1"
-AR Path="/616EB94F/616F9E75" Ref="U?"  Part="1"
-F 0 "U?" H 3400 3183 50  0000 C CNN
-F 1 "LM358" H 3400 3274 50  0000 C CNN
-F 2 "" H 3400 3550 50  0001 C CNN
-F 3 "http://www.ti.com/lit/ds/symlink/lm2904-n.pdf" H 3400 3550 50  0001 C CNN
-	1    3400 3550
-	1    0    0    1
-$EndComp
 $Comp
 L Device:R_US R?
@@
 Text Label 3850 3550 0    50   ~ 0
 freq_sel_v
-$Comp
-L 2021-10-12_02-33-31:TLC555CP U?
-U 1 1 616F9EDC
-P 5900 3700
-AR Path="/616F9EDC" Ref="U?"  Part="1"
-AR Path="/616EB94F/616F9EDC" Ref="U?"  Part="1"
-F 0 "U?" H 5900 4488 60  0000 C CNN
-F 1 "TLC555CP" H 5900 4382 60  0000 C CNN
-F 2 "P0008A" H 5900 3640 60  0001 C CNN
-F 3 "" H 5900 3700 60  0000 C CNN
-	1    5900 3700
-	1    0    0    -1
-$EndComp
 Wire Wire Line
 	5200 3900 5100 3900
@@
 square_out
 $Comp
-L SimpleArduinoVlfRadio-rescue:MAX292-Custom_Library U?
-U 1 1 617C60A4
-P 8200 3100
-F 0 "U?" H 8200 3175 50  0000 C CNN
-F 1 "MAX292-Custom_Library" H 8200 3084 50  0000 C CNN
-F 2 "" H 8200 3000 50  0001 C CNN
-F 3 "" H 8200 3000 50  0001 C CNN
-	1    8200 3100
-	1    0    0    -1
-$EndComp
-$Comp
 L Device:C C?
 U 1 1 617CD1E2
@@
 Wire Wire Line
 	7650 3700 7750 3700
+$Comp
+L 2021-10-12_02-33-31:TLC555CP U?
+U 1 1 616F9EDC
+P 5900 3700
+AR Path="/616F9EDC" Ref="U?"  Part="1"
+AR Path="/616EB94F/616F9EDC" Ref="U2"  Part="1"
+F 0 "U2" H 5900 4488 60  0000 C CNN
+F 1 "555" H 5900 4382 60  0000 C CNN
+F 2 "" H 5900 3640 60  0001 C CNN
+F 3 "http://www.ti.com/lit/ds/symlink/lm2904-n.pdf" H 5900 3700 60  0000 C CNN
+	1    5900 3700
+	1    0    0    -1
+$EndComp
+$Comp
+L SimpleArduinoVlfRadio-rescue:MAX292-Custom_Library U3
+U 1 1 617C60A4
+P 8200 3100
+F 0 "U3" H 8200 3175 50  0000 C CNN
+F 1 "MAX292" H 8200 3084 50  0000 C CNN
+F 2 "" H 8200 3000 50  0001 C CNN
+F 3 "http://www.ti.com/lit/ds/symlink/lm2904-n.pdf" H 8200 3000 50  0001 C CNN
+	1    8200 3100
+	1    0    0    -1
+$EndComp
+$Comp
+L Amplifier_Operational:LM358 U?
+U 1 1 616F9E75
+P 3400 3550
+AR Path="/616F9E75" Ref="U?"  Part="1"
+AR Path="/616EB94F/616F9E75" Ref="U1"  Part="1"
+F 0 "U1" H 3400 3183 50  0000 C CNN
+F 1 "LM358" H 3400 3274 50  0000 C CNN
+F 2 "" H 3400 3550 50  0001 C CNN
+F 3 "http://www.ti.com/lit/ds/symlink/lm2904-n.pdf" H 3400 3550 50  0001 C CNN
+	1    3400 3550
+	1    0    0    1
+$EndComp
 $EndSCHEMATC
